Commit message: fixed errors to load cpp

File: bimanual_ws/src/Bimanual_Robot_Project_MuJoCo/urdf/bimanual_panda.urdf.xacro (robot description, xacro)
@@ -19,20 +19,52 @@
   </link>
   <xacro:panda_arm arm_id="left" connected_to="base" xyz="0 0.5 1" safety_distance="0.03"/>
-  <xacro:hand arm_id="left" rpy="0 0 ${-pi/4}" connected_to="left_link8" safety_distance="0.03"/>
-  <xacro:gazebo-joint joint="left_joint1" transmission="hardware_interface/PositionJointInterface" />
-  <xacro:gazebo-joint joint="left_joint2" transmission="hardware_interface/PositionJointInterface" />
-  <xacro:gazebo-joint joint="left_joint3" transmission="hardware_interface/PositionJointInterface" />
-  <xacro:gazebo-joint joint="left_joint4" transmission="hardware_interface/PositionJointInterface" />
-  <xacro:gazebo-joint joint="left_joint5" transmission="hardware_interface/PositionJointInterface" />
-  <xacro:gazebo-joint joint="left_joint6" transmission="hardware_interface/PositionJointInterface" />
-  <xacro:gazebo-joint joint="left_joint7" transmission="hardware_interface/PositionJointInterface" />
-  <xacro:panda_arm arm_id="right" connected_to="base" xyz="0 -0.5 1" safety_distance="0.03"/>
-  <xacro:hand arm_id="right" rpy="0 0 ${-pi/4}" connected_to="right_link8" safety_distance="0.03"/>
-  <xacro:gazebo-joint joint="right_joint1" transmission="hardware_interface/PositionJointInterface" />
-  <xacro:gazebo-joint joint="right_joint2" transmission="hardware_interface/PositionJointInterface" />
-  <xacro:gazebo-joint joint="right_joint3" transmission="hardware_interface/PositionJointInterface" />
-  <xacro:gazebo-joint joint="right_joint4" transmission="hardware_interface/PositionJointInterface" />
-  <xacro:gazebo-joint joint="right_joint5" transmission="hardware_interface/PositionJointInterface" />
-  <xacro:gazebo-joint joint="right_joint6" transmission="hardware_interface/PositionJointInterface" />
-  <xacro:gazebo-joint joint="right_joint7" transmission="hardware_interface/PositionJointInterface" />
+<xacro:hand arm_id="left" rpy="0 0 ${-pi/4}" connected_to="left_link8" safety_distance="0.03"/>
+<xacro:gazebo-joint joint="left_joint1" transmission="hardware_interface/PositionJointInterface" />
+<xacro:gazebo-joint joint="left_joint2" transmission="hardware_interface/PositionJointInterface" />
+<xacro:gazebo-joint joint="left_joint3" transmission="hardware_interface/PositionJointInterface" />
+<xacro:gazebo-joint joint="left_joint4" transmission="hardware_interface/PositionJointInterface" />
+<xacro:gazebo-joint joint="left_joint5" transmission="hardware_interface/PositionJointInterface" />
+<xacro:gazebo-joint joint="left_joint6" transmission="hardware_interface/PositionJointInterface" />
+<xacro:gazebo-joint joint="left_joint7" transmission="hardware_interface/PositionJointInterface" />
+<xacro:gazebo-joint joint="left_joint1" transmission="hardware_interface/VelocityJointInterface" />
+<xacro:gazebo-joint joint="left_joint2" transmission="hardware_interface/VelocityJointInterface" />
+<xacro:gazebo-joint joint="left_joint3" transmission="hardware_interface/VelocityJointInterface" />
+<xacro:gazebo-joint joint="left_joint4" transmission="hardware_interface/VelocityJointInterface" />
+<xacro:gazebo-joint joint="left_joint5" transmission="hardware_interface/VelocityJointInterface" />
+<xacro:gazebo-joint joint="left_joint6" transmission="hardware_interface/VelocityJointInterface" />
+<xacro:gazebo-joint joint="left_joint7" transmission="hardware_interface/VelocityJointInterface" />
+<xacro:gazebo-joint joint="left_joint1" transmission="hardware_interface/EffortJointInterface" />
+<xacro:gazebo-joint joint="left_joint2" transmission="hardware_interface/EffortJointInterface" />
+<xacro:gazebo-joint joint="left_joint3" transmission="hardware_interface/EffortJointInterface" />
+<xacro:gazebo-joint joint="left_joint4" transmission="hardware_interface/EffortJointInterface" />
+<xacro:gazebo-joint joint="left_joint5" transmission="hardware_interface/EffortJointInterface" />
+<xacro:gazebo-joint joint="left_joint6" transmission="hardware_interface/EffortJointInterface" />
+<xacro:gazebo-joint joint="left_joint7" transmission="hardware_interface/EffortJointInterface" />
+<xacro:transmission-franka-state arm_id="left" />
+<xacro:transmission-franka-model arm_id="left" root="left_joint1" tip="left_joint8" />
+<xacro:panda_arm arm_id="right" connected_to="base" xyz="0 -0.5 1" safety_distance="0.03"/>
+<xacro:hand arm_id="right" rpy="0 0 ${-pi/4}" connected_to="right_link8" safety_distance="0.03"/>
+<xacro:gazebo-joint joint="right_joint1" transmission="hardware_interface/PositionJointInterface" />
+<xacro:gazebo-joint joint="right_joint2" transmission="hardware_interface/PositionJointInterface" />
+<xacro:gazebo-joint joint="right_joint3" transmission="hardware_interface/PositionJointInterface" />
+<xacro:gazebo-joint joint="right_joint4" transmission="hardware_interface/PositionJointInterface" />
+<xacro:gazebo-joint joint="right_joint5" transmission="hardware_interface/PositionJointInterface" />
+<xacro:gazebo-joint joint="right_joint6" transmission="hardware_interface/PositionJointInterface" />
+<xacro:gazebo-joint joint="right_joint7" transmission="hardware_interface/PositionJointInterface" />
+<xacro:gazebo-joint joint="right_joint1" transmission="hardware_interface/VelocityJointInterface" />
+<xacro:gazebo-joint joint="right_joint2" transmission="hardware_interface/VelocityJointInterface" />
+<xacro:gazebo-joint joint="right_joint3" transmission="hardware_interface/VelocityJointInterface" />
+<xacro:gazebo-joint joint="right_joint4" transmission="hardware_interface/VelocityJointInterface" />
+<xacro:gazebo-joint joint="right_joint5" transmission="hardware_interface/VelocityJointInterface" />
+<xacro:gazebo-joint joint="right_joint6" transmission="hardware_interface/VelocityJointInterface" />
+<xacro:gazebo-joint joint="right_joint7" transmission="hardware_interface/VelocityJointInterface" />
+<xacro:gazebo-joint joint="right_joint1" transmission="hardware_interface/EffortJointInterface" />
+<xacro:gazebo-joint joint="right_joint2" transmission="hardware_interface/EffortJointInterface" />
+<xacro:gazebo-joint joint="right_joint3" transmission="hardware_interface/EffortJointInterface" />
+<xacro:gazebo-joint joint="right_joint4" transmission="hardware_interface/EffortJointInterface" />
+<xacro:gazebo-joint joint="right_joint5" transmission="hardware_interface/EffortJointInterface" />
+<xacro:gazebo-joint joint="right_joint6" transmission="hardware_interface/EffortJointInterface" />
+<xacro:gazebo-joint joint="right_joint7" transmission="hardware_interface/EffortJointInterface" />
+<xacro:transmission-franka-state arm_id="right" />
+<xacro:transmission-franka-model arm_id="right" root="right_joint1" tip="right_joint8" />
 </robot>

File: bimanual_ws/src/franka_ros/franka_description/robots/hand.urdf.xacro (robot description, xacro)
@@ -1,5 +1,4 @@
 <?xml version="1.0" encoding="utf-8"?>
 <robot xmlns:xacro="http://www.ros.org/wiki/xacro" name="hand">
-  <xacro:include filename="utils.xacro" />
   <xacro:include filename="hand.xacro"/>
   <xacro:hand arm_id="panda" safety_distance="0.03"/>

File: bimanual_ws/src/franka_ros/franka_description/robots/hand.xacro (robot description, xacro)
@@ -2,22 +2,59 @@
 <robot xmlns:xacro="http://www.ros.org/wiki/xacro" name="hand">
   <!-- safety_distance: Minimum safety distance in [m] by which the collision volumes are expanded and which is enforced during robot motions -->
-  <xacro:macro name="hand" params="connected_to:='' arm_id:='panda' rpy:='0 0 0' xyz:='0 0 0' tcp_xyz:='0 0 0.1034' tcp_rpy:='0 0 0' safety_distance:=0 gazebo:=false description_pkg:=franka_description">
+  <xacro:macro name="hand" params="connected_to:='' arm_id:='panda' rpy:='0 0 0' xyz:='0 0 0' safety_distance:=0">
     <xacro:unless value="${connected_to == ''}">
       <joint name="${arm_id}_hand_joint" type="fixed">
-        <parent link="${connected_to}" />
-        <child link="${arm_id}_hand" />
-        <origin xyz="${xyz}" rpy="${rpy}" />
+        <parent link="${connected_to}"/>
+        <child link="${arm_id}_hand"/>
+        <origin xyz="${xyz}" rpy="${rpy}"/>
       </joint>
     </xacro:unless>
-    <xacro:link_with_sc name="hand" gazebo="${gazebo}">
-      <self_collision_geometries>
-        <xacro:collision_capsule xyz="0 0 0.04" direction="y" radius="${0.04+safety_distance}" length="0.1" />
-        <xacro:collision_capsule xyz="0 0 0.10" direction="y" radius="${0.02+safety_distance}" length="0.1" />
-      </self_collision_geometries>
-    </xacro:link_with_sc>
+    <link name="${arm_id}_hand">
+      <visual>
+        <geometry>
+          <mesh filename="package://franka_description/meshes/visual/hand.dae"/>
+        </geometry>
+      </visual>
+      <collision>
+        <origin xyz="0 0 0.04" rpy="0 ${pi/2} ${pi/2}"/>
+        <geometry>
+          <cylinder radius="${0.04+safety_distance}" length="0.1" />
+        </geometry>
+      </collision>
+      <collision>
+        <origin xyz="0 -0.05 0.04" rpy="0 0 0"/>
+        <geometry>
+          <sphere radius="${0.04+safety_distance}"  />
+        </geometry>
+      </collision>
+      <collision>
+        <origin xyz="0 0.05 0.04" rpy="0 0 0"/>
+        <geometry>
+          <sphere radius="${0.04+safety_distance}"  />
+        </geometry>
+      </collision>
+      <collision>
+        <origin xyz="0 0 0.1" rpy="0 ${pi/2} ${pi/2}"/>
+        <geometry>
+          <cylinder radius="${0.02+safety_distance}" length="0.1" />
+        </geometry>
+      </collision>
+      <collision>
+        <origin xyz="0 -0.05 0.1" rpy="0 0 0"/>
+        <geometry>
+          <sphere radius="${0.02+safety_distance}"  />
+        </geometry>
+      </collision>
+      <collision>
+        <origin xyz="0 0.05 0.1" rpy="0 0 0"/>
+        <geometry>
+          <sphere radius="${0.02+safety_distance}"  />
+        </geometry>
+      </collision>
+    </link>
     <!-- Define the hand_tcp frame -->
     <link name="${arm_id}_hand_tcp" />
     <joint name="${arm_id}_hand_tcp_joint" type="fixed">
-      <origin xyz="${tcp_xyz}" rpy="${tcp_rpy}" />
+      <origin xyz="0 0 0.1034" rpy="0 0 0" />
       <parent link="${arm_id}_hand" />
       <child link="${arm_id}_hand_tcp" />
@@ -26,94 +63,30 @@
       <visual>
         <geometry>
-          <mesh filename="package://${description_pkg}/meshes/visual/finger.dae" />
+          <mesh filename="package://franka_description/meshes/visual/finger.dae"/>
         </geometry>
       </visual>
-      <!-- screw mount -->
-      <collision>
-        <origin xyz="0 18.5e-3 11e-3" rpy="0 0 0" />
-        <geometry>
-          <box size="22e-3 15e-3 20e-3" />
-        </geometry>
-      </collision>
-      <!-- cartriage sledge -->
-      <collision>
-        <origin xyz="0 6.8e-3 2.2e-3" rpy="0 0 0" />
-        <geometry>
-          <box size="22e-3 8.8e-3 3.8e-3" />
-        </geometry>
-      </collision>
-      <!-- diagonal finger -->
-      <collision>
-        <origin xyz="0 15.9e-3 28.35e-3" rpy="${pi/6} 0 0" />
-        <geometry>
-          <box size="17.5e-3 7e-3 23.5e-3" />
-        </geometry>
-      </collision>
-      <!-- rubber tip with which to grasp -->
-      <collision>
-        <origin xyz="0 7.58e-3 45.25e-3" rpy="0 0 0" />
-        <geometry>
-          <box size="17.5e-3 15.2e-3 18.5e-3" />
-        </geometry>
-      </collision>
-      <xacro:if value="${gazebo}">
-        <xacro:inertial_props name="leftfinger" />
-      </xacro:if>
     </link>
     <link name="${arm_id}_rightfinger">
       <visual>
-        <origin xyz="0 0 0" rpy="0 0 ${pi}" />
+        <origin xyz="0 0 0" rpy="0 0 ${pi}"/>
         <geometry>
-          <mesh filename="package://${description_pkg}/meshes/visual/finger.dae" />
+          <mesh filename="package://franka_description/meshes/visual/finger.dae"/>
         </geometry>
       </visual>
-      <!-- screw mount -->
-      <collision>
-        <origin xyz="0 -18.5e-3 11e-3" rpy="0 0 0" />
-        <geometry>
-          <box size="22e-3 15e-3 20e-3" />
-        </geometry>
-      </collision>
-      <!-- cartriage sledge -->
-      <collision>
-        <origin xyz="0 -6.8e-3 2.2e-3" rpy="0 0 0" />
-        <geometry>
-          <box size="22e-3 8.8e-3 3.8e-3" />
-        </geometry>
-      </collision>
-      <!-- diagonal finger -->
-      <collision>
-        <origin xyz="0 -15.9e-3 28.35e-3" rpy="${-pi/6} 0 0" />
-        <geometry>
-          <box size="17.5e-3 7e-3 23.5e-3" />
-        </geometry>
-      </collision>
-      <!-- rubber tip with which to grasp -->
-      <collision>
-        <origin xyz="0 -7.58e-3 45.25e-3" rpy="0 0 0" />
-        <geometry>
-          <box size="17.5e-3 15.2e-3 18.5e-3" />
-        </geometry>
-      </collision>
-      <xacro:if value="${gazebo}">
-        <xacro:inertial_props name="rightfinger" />
-      </xacro:if>
-    </link>
+   </link>
     <joint name="${arm_id}_finger_joint1" type="prismatic">
-      <parent link="${arm_id}_hand" />
-      <child link="${arm_id}_leftfinger" />
-      <origin xyz="0 0 0.0584" rpy="0 0 0" />
-      <axis xyz="0 1 0" />
-      <limit effort="100" lower="0.0" upper="0.04" velocity="0.2" />
-      <dynamics damping="0.3" />
+      <parent link="${arm_id}_hand"/>
+      <child link="${arm_id}_leftfinger"/>
+      <origin xyz="0 0 0.0584" rpy="0 0 0"/>
+      <axis xyz="0 1 0"/>
+      <limit effort="100" lower="0.0" upper="0.04" velocity="0.2"/>
     </joint>
     <joint name="${arm_id}_finger_joint2" type="prismatic">
-      <parent link="${arm_id}_hand" />
-      <child link="${arm_id}_rightfinger" />
-      <origin xyz="0 0 0.0584" rpy="0 0 0" />
-      <axis xyz="0 -1 0" />
-      <limit effort="100" lower="0.0" upper="0.04" velocity="0.2" />
+      <parent link="${arm_id}_hand"/>
+      <child link="${arm_id}_rightfinger"/>
+      <origin xyz="0 0 0.0584" rpy="0 0 0"/>
+      <axis xyz="0 -1 0"/>
+      <limit effort="100" lower="0.0" upper="0.04" velocity="0.2"/>
       <mimic joint="${arm_id}_finger_joint1" />
-      <dynamics damping="0.3" />
     </joint>
   </xacro:macro>

File: bimanual_ws/src/franka_ros/franka_description/robots/panda_arm.urdf.xacro (robot description, xacro)
@@ -5,29 +5,27 @@
   <!-- Should a franka_gripper be mounted at the flange?" -->
   <xacro:arg name="hand" default="false" />
-  <!-- Positional offset between $(arm_id)_hand -> $(arm_id)_hand_tcp [m]. Only used when hand:=true -->
-  <xacro:arg name="tcp_xyz" default="0 0 0.1034" />
-  <!-- Rotational offset between $(arm_id)_hand -> $(arm_id)_hand_tcp [rad]. Only used when hand:=true -->
-  <xacro:arg name="tcp_rpy" default="0 0 0" />
   <!-- Is the robot being simulated in gazebo?" -->
   <xacro:arg name="gazebo" default="false" />
-  <xacro:include filename="utils.xacro" />
-  <xacro:include filename="panda_arm.xacro" />
-  <xacro:panda_arm arm_id="$(arg arm_id)" safety_distance="0.03" gazebo="$(arg gazebo)"/>
-  <xacro:if value="$(arg hand)">
-    <xacro:include filename="hand.xacro"/>
-    <xacro:hand
-        arm_id="$(arg arm_id)"
-        rpy="0 0 ${-pi/4}"
-        tcp_xyz="$(arg tcp_xyz)"
-        tcp_rpy="$(arg tcp_rpy)"
-        connected_to="$(arg arm_id)_link8"
-        safety_distance="0.03"
-        gazebo="$(arg gazebo)"
-     />
-  </xacro:if>
-  <!-- Define additional Gazebo tags -->
+  <xacro:unless value="$(arg gazebo)">
+    <!-- Create a URDF for a real hardware -->
+    <xacro:include filename="$(find franka_description)/robots/panda_arm.xacro" />
+    <xacro:panda_arm arm_id="$(arg arm_id)" safety_distance="0.03"/>
+    <xacro:if value="$(arg hand)">
+      <xacro:include filename="$(find franka_description)/robots/hand.xacro"/>
+      <xacro:hand arm_id="$(arg arm_id)" rpy="0 0 ${-pi/4}" connected_to="$(arg arm_id)_link8" safety_distance="0.03"/>
+    </xacro:if>
+  </xacro:unless>
   <xacro:if value="$(arg gazebo)">
     <xacro:arg name="xyz" default="0 0 0" />
     <xacro:arg name="rpy" default="0 0 0" />
+    <!-- Create a simulatable URDF -->
+    <xacro:include filename="$(find franka_description)/robots/utils.xacro" />
+    <xacro:include filename="$(find franka_description)/robots/panda_gazebo.xacro" />
+    <xacro:panda_arm arm_id="$(arg arm_id)" />
+    <xacro:if value="$(arg hand)">
+      <xacro:hand arm_id="$(arg arm_id)" rpy="0 0 ${-pi/4}" connected_to="$(arg arm_id)_link8" />
+      <xacro:gazebo-joint joint="$(arg arm_id)_finger_joint1" transmission="hardware_interface/EffortJointInterface" />
+      <xacro:gazebo-joint joint="$(arg arm_id)_finger_joint2" transmission="hardware_interface/EffortJointInterface" />
+    </xacro:if>
     <!-- Gazebo requires a joint to a link called "world" for statically mounted robots -->
     <link name="world" />
@@ -63,11 +61,4 @@
        tip="$(arg arm_id)_joint8"
      />
-    <xacro:if value="$(arg hand)">
-      <xacro:gazebo-joint joint="$(arg arm_id)_finger_joint1" transmission="hardware_interface/EffortJointInterface" />
-      <xacro:gazebo-joint joint="$(arg arm_id)_finger_joint2" transmission="hardware_interface/EffortJointInterface" />
-      <!-- Friction specific material for Rubber/Rubber contact -->
-      <xacro:gazebo-friction link="$(arg arm_id)_leftfinger" mu="1.13" />
-      <xacro:gazebo-friction link="$(arg arm_id)_rightfinger" mu="1.13" />
-    </xacro:if>
     <gazebo>
       <plugin name="gazebo_ros_control" filename="libgazebo_ros_control.so">
